File: 65_keyboard/65_keyboard.kicad_pcb (KiCad board)
At the start: 2 copper layers, 10 parts, among them SW0-0 MX, SW1-0 MX, SW2-0 MX, SW3-0 MX, SW4-0 MX

Commit message: Adds all keys to keyboard, and places them on the PCB
Parts:
- added D0-1: D, Diodes_ThroughHole:Diode_DO-35_SOD27_Horizontal_RM10, B.Cu at (73.8, 116.7)
- added D0-10: D, Diodes_ThroughHole:Diode_DO-35_SOD27_Horizontal_RM10, B.Cu at (245.3, 116.7)
- added D0-11: D, Diodes_ThroughHole:Diode_DO-35_SOD27_Horizontal_RM10, B.Cu at (264.3, 116.7)
- added D0-12: D, Diodes_ThroughHole:Diode_DO-35_SOD27_Horizontal_RM10, B.Cu at (283.4, 116.7)
- added D0-14: D, Diodes_ThroughHole:Diode_DO-35_SOD27_Horizontal_RM10, B.Cu at (311.9, 116.7)
- added D0-15: D, Diodes_ThroughHole:Diode_DO-35_SOD27_Horizontal_RM10, B.Cu at (340.5, 116.7)
- added D0-2: D, Diodes_ThroughHole:Diode_DO-35_SOD27_Horizontal_RM10, B.Cu at (92.9, 116.7)
- added D0-3: D, Diodes_ThroughHole:Diode_DO-35_SOD27_Horizontal_RM10, B.Cu at (111.9, 116.7)
- added D0-4: D, Diodes_ThroughHole:Diode_DO-35_SOD27_Horizontal_RM10, B.Cu at (131.0, 116.7)
- added D0-5: D, Diodes_ThroughHole:Diode_DO-35_SOD27_Horizontal_RM10, B.Cu at (150.0, 116.7)
- added D0-6: D, Diodes_ThroughHole:Diode_DO-35_SOD27_Horizontal_RM10, B.Cu at (169.1, 116.7)
- added D0-7: D, Diodes_ThroughHole:Diode_DO-35_SOD27_Horizontal_RM10, B.Cu at (188.1, 116.7)
- added D0-8: D, Diodes_ThroughHole:Diode_DO-35_SOD27_Horizontal_RM10, B.Cu at (207.2, 116.7)
- added D0-9: D, Diodes_ThroughHole:Diode_DO-35_SOD27_Horizontal_RM10, B.Cu at (226.2, 116.7)
- added D1-1: D, Diodes_ThroughHole:Diode_DO-35_SOD27_Horizontal_RM10, B.Cu at (83.3, 135.7)
- added D1-10: D, Diodes_ThroughHole:Diode_DO-35_SOD27_Horizontal_RM10, B.Cu at (254.8, 135.7)
- added D1-11: D, Diodes_ThroughHole:Diode_DO-35_SOD27_Horizontal_RM10, B.Cu at (273.8, 135.7)
- added D1-12: D, Diodes_ThroughHole:Diode_DO-35_SOD27_Horizontal_RM10, B.Cu at (292.9, 135.7)
- added D1-14: D, Diodes_ThroughHole:Diode_DO-35_SOD27_Horizontal_RM10, B.Cu at (316.7, 135.7)
- added D1-15: D, Diodes_ThroughHole:Diode_DO-35_SOD27_Horizontal_RM10, B.Cu at (340.5, 135.7)
- added D1-2: D, Diodes_ThroughHole:Diode_DO-35_SOD27_Horizontal_RM10, B.Cu at (102.4, 135.7)
- added D1-3: D, Diodes_ThroughHole:Diode_DO-35_SOD27_Horizontal_RM10, B.Cu at (121.4, 135.7)
- added D1-4: D, Diodes_ThroughHole:Diode_DO-35_SOD27_Horizontal_RM10, B.Cu at (140.5, 135.7)
- added D1-5: D, Diodes_ThroughHole:Diode_DO-35_SOD27_Horizontal_RM10, B.Cu at (159.5, 135.7)
- added D1-6: D, Diodes_ThroughHole:Diode_DO-35_SOD27_Horizontal_RM10, B.Cu at (178.6, 135.7)
- added D1-7: D, Diodes_ThroughHole:Diode_DO-35_SOD27_Horizontal_RM10, B.Cu at (197.6, 135.7)
- added D1-8: D, Diodes_ThroughHole:Diode_DO-35_SOD27_Horizontal_RM10, B.Cu at (216.7, 135.7)
- added D1-9: D, Diodes_ThroughHole:Diode_DO-35_SOD27_Horizontal_RM10, B.Cu at (235.7, 135.7)
- added D2-1: D, Diodes_ThroughHole:Diode_DO-35_SOD27_Horizontal_RM10, B.Cu at (88.1, 154.8)
- added D2-10: D, Diodes_ThroughHole:Diode_DO-35_SOD27_Horizontal_RM10, B.Cu at (259.6, 154.8)
- added D2-11: D, Diodes_ThroughHole:Diode_DO-35_SOD27_Horizontal_RM10, B.Cu at (278.6, 154.8)
- added D2-14: D, Diodes_ThroughHole:Diode_DO-35_SOD27_Horizontal_RM10, B.Cu at (309.6, 154.8)
- added D2-15: D, Diodes_ThroughHole:Diode_DO-35_SOD27_Horizontal_RM10, B.Cu at (340.5, 154.8)
- added D2-2: D, Diodes_ThroughHole:Diode_DO-35_SOD27_Horizontal_RM10, B.Cu at (107.2, 154.8)
- added D2-3: D, Diodes_ThroughHole:Diode_DO-35_SOD27_Horizontal_RM10, B.Cu at (126.2, 154.8)
- added D2-4: D, Diodes_ThroughHole:Diode_DO-35_SOD27_Horizontal_RM10, B.Cu at (145.3, 154.8)
- added D2-5: D, Diodes_ThroughHole:Diode_DO-35_SOD27_Horizontal_RM10, B.Cu at (164.3, 154.8)
- added D2-6: D, Diodes_ThroughHole:Diode_DO-35_SOD27_Horizontal_RM10, B.Cu at (183.4, 154.8)
- added D2-7: D, Diodes_ThroughHole:Diode_DO-35_SOD27_Horizontal_RM10, B.Cu at (202.4, 154.8)
- added D2-8: D, Diodes_ThroughHole:Diode_DO-35_SOD27_Horizontal_RM10, B.Cu at (221.5, 154.8)
- added D2-9: D, Diodes_ThroughHole:Diode_DO-35_SOD27_Horizontal_RM10, B.Cu at (240.5, 154.8)
- added D3-10: D, Diodes_ThroughHole:Diode_DO-35_SOD27_Horizontal_RM10, B.Cu at (250.0, 173.8)
- added D3-11: D, Diodes_ThroughHole:Diode_DO-35_SOD27_Horizontal_RM10, B.Cu at (269.1, 173.8)
- added D3-13: D, Diodes_ThroughHole:Diode_DO-35_SOD27_Horizontal_RM10, B.Cu at (295.3, 173.8)
- added D3-14: D, Diodes_ThroughHole:Diode_DO-35_SOD27_Horizontal_RM10, B.Cu at (321.5, 173.8)
- added D3-15: D, Diodes_ThroughHole:Diode_DO-35_SOD27_Horizontal_RM10, B.Cu at (340.5, 173.8)
- added D3-2: D, Diodes_ThroughHole:Diode_DO-35_SOD27_Horizontal_RM10, B.Cu at (97.6, 173.8)
- added D3-3: D, Diodes_ThroughHole:Diode_DO-35_SOD27_Horizontal_RM10, B.Cu at (116.7, 173.8)
- added D3-4: D, Diodes_ThroughHole:Diode_DO-35_SOD27_Horizontal_RM10, B.Cu at (135.7, 173.8)
- added D3-5: D, Diodes_ThroughHole:Diode_DO-35_SOD27_Horizontal_RM10, B.Cu at (154.8, 173.8)
- added D3-6: D, Diodes_ThroughHole:Diode_DO-35_SOD27_Horizontal_RM10, B.Cu at (173.8, 173.8)
- added D3-7: D, Diodes_ThroughHole:Diode_DO-35_SOD27_Horizontal_RM10, B.Cu at (192.9, 173.8)
- added D3-8: D, Diodes_ThroughHole:Diode_DO-35_SOD27_Horizontal_RM10, B.Cu at (211.9, 173.8)
- added D3-9: D, Diodes_ThroughHole:Diode_DO-35_SOD27_Horizontal_RM10, B.Cu at (231.0, 173.8)
- added D4-10: D, Diodes_ThroughHole:Diode_DO-35_SOD27_Horizontal_RM10, B.Cu at (238.1, 192.9)
- added D4-11: D, Diodes_ThroughHole:Diode_DO-35_SOD27_Horizontal_RM10, B.Cu at (259.6, 192.9)
- added D4-12: D, Diodes_ThroughHole:Diode_DO-35_SOD27_Horizontal_RM10, B.Cu at (281.0, 192.9)
- added D4-13: D, Diodes_ThroughHole:Diode_DO-35_SOD27_Horizontal_RM10, B.Cu at (302.4, 192.9)
- added D4-14: D, Diodes_ThroughHole:Diode_DO-35_SOD27_Horizontal_RM10, B.Cu at (321.5, 192.9)
- added D4-15: D, Diodes_ThroughHole:Diode_DO-35_SOD27_Horizontal_RM10, B.Cu at (340.5, 192.9)
- added D4-2: D, Diodes_ThroughHole:Diode_DO-35_SOD27_Horizontal_RM10, B.Cu at (92.9, 192.9)
- added D4-7: D, Diodes_ThroughHole:Diode_DO-35_SOD27_Horizontal_RM10, B.Cu at (166.7, 192.9)
- added SW0-1: MX, Keyboard:CHERRY_PLATE_100H, F.Cu at (78.6, 109.5)
- added SW0-10: MX, Keyboard:CHERRY_PLATE_100H, F.Cu at (250.0, 109.5)
- added SW0-11: MX, Keyboard:CHERRY_PLATE_100H, F.Cu at (269.1, 109.5)
- added SW0-12: MX, Keyboard:CHERRY_PLATE_100H, F.Cu at (288.1, 109.5)
- added SW0-14: MX, Keyboard:CHERRY_PLATE_200H, F.Cu at (316.7, 109.5)
- added SW0-15: MX, Keyboard:CHERRY_PLATE_100H, F.Cu at (345.3, 109.5)
- added SW0-2: MX, Keyboard:CHERRY_PLATE_100H, F.Cu at (97.6, 109.5)
- added SW0-3: MX, Keyboard:CHERRY_PLATE_100H, F.Cu at (116.7, 109.5)
- added SW0-4: MX, Keyboard:CHERRY_PLATE_100H, F.Cu at (135.7, 109.5)
- added SW0-5: MX, Keyboard:CHERRY_PLATE_100H, F.Cu at (154.8, 109.5)
- added SW0-6: MX, Keyboard:CHERRY_PLATE_100H, F.Cu at (173.8, 109.5)
- added SW0-7: MX, Keyboard:CHERRY_PLATE_100H, F.Cu at (192.9, 109.5)
- added SW0-8: MX, Keyboard:CHERRY_PLATE_100H, F.Cu at (211.9, 109.5)
- added SW0-9: MX, Keyboard:CHERRY_PLATE_100H, F.Cu at (231.0, 109.5)
- added SW1-1: MX, Keyboard:CHERRY_PLATE_100H, F.Cu at (88.1, 128.6)
- added SW1-10: MX, Keyboard:CHERRY_PLATE_100H, F.Cu at (259.6, 128.6)
- added SW1-11: MX, Keyboard:CHERRY_PLATE_100H, F.Cu at (278.6, 128.6)
- added SW1-12: MX, Keyboard:CHERRY_PLATE_100H, F.Cu at (297.7, 128.6)
- added SW1-14: MX, Keyboard:CHERRY_PLATE_150H, F.Cu at (321.5, 128.6)
- added SW1-15: MX, Keyboard:CHERRY_PLATE_100H, F.Cu at (345.3, 128.6)
- added SW1-2: MX, Keyboard:CHERRY_PLATE_100H, F.Cu at (107.2, 128.6)
- added SW1-3: MX, Keyboard:CHERRY_PLATE_100H, F.Cu at (126.2, 128.6)
- added SW1-4: MX, Keyboard:CHERRY_PLATE_100H, F.Cu at (145.3, 128.6)
- added SW1-5: MX, Keyboard:CHERRY_PLATE_100H, F.Cu at (164.3, 128.6)
- added SW1-6: MX, Keyboard:CHERRY_PLATE_100H, F.Cu at (183.4, 128.6)
- added SW1-7: MX, Keyboard:CHERRY_PLATE_100H, F.Cu at (202.4, 128.6)
- added SW1-8: MX, Keyboard:CHERRY_PLATE_100H, F.Cu at (221.5, 128.6)
- added SW1-9: MX, Keyboard:CHERRY_PLATE_100H, F.Cu at (240.5, 128.6)
- added SW2-1: MX, Keyboard:CHERRY_PLATE_100H, F.Cu at (92.9, 147.6)
- added SW2-10: MX, Keyboard:CHERRY_PLATE_100H, F.Cu at (264.3, 147.6)
- added SW2-11: MX, Keyboard:CHERRY_PLATE_100H, F.Cu at (283.4, 147.6)
- added SW2-14: MX, Keyboard:CHERRY_PLATE_225H, F.Cu at (314.3, 147.6)
- added SW2-15: MX, Keyboard:CHERRY_PLATE_100H, F.Cu at (345.3, 147.6)
- added SW2-2: MX, Keyboard:CHERRY_PLATE_100H, F.Cu at (111.9, 147.6)
- added SW2-3: MX, Keyboard:CHERRY_PLATE_100H, F.Cu at (131.0, 147.6)
- added SW2-4: MX, Keyboard:CHERRY_PLATE_100H, F.Cu at (150.0, 147.6)
- added SW2-5: MX, Keyboard:CHERRY_PLATE_100H, F.Cu at (169.1, 147.6)
- added SW2-6: MX, Keyboard:CHERRY_PLATE_100H, F.Cu at (188.1, 147.6)
- added SW2-7: MX, Keyboard:CHERRY_PLATE_100H, F.Cu at (207.2, 147.6)
- added SW2-8: MX, Keyboard:CHERRY_PLATE_100H, F.Cu at (226.2, 147.6)
- added SW2-9: MX, Keyboard:CHERRY_PLATE_100H, F.Cu at (245.3, 147.6)
- added SW3-10: MX, Keyboard:CHERRY_PLATE_100H, F.Cu at (254.8, 166.7)
- added SW3-11: MX, Keyboard:CHERRY_PLATE_100H, F.Cu at (273.8, 166.7)
- added SW3-13: MX, Keyboard:CHERRY_PLATE_175H, F.Cu at (300.0, 166.7)
- added SW3-14: MX, Keyboard:CHERRY_PLATE_100H, F.Cu at (326.2, 166.7)
- added SW3-15: MX, Keyboard:CHERRY_PLATE_100H, F.Cu at (345.3, 166.7)
- added SW3-2: MX, Keyboard:CHERRY_PLATE_100H, F.Cu at (102.4, 166.7)
- added SW3-3: MX, Keyboard:CHERRY_PLATE_100H, F.Cu at (121.4, 166.7)
- added SW3-4: MX, Keyboard:CHERRY_PLATE_100H, F.Cu at (140.5, 166.7)
- added SW3-5: MX, Keyboard:CHERRY_PLATE_100H, F.Cu at (159.5, 166.7)
- added SW3-6: MX, Keyboard:CHERRY_PLATE_100H, F.Cu at (178.6, 166.7)
- added SW3-7: MX, Keyboard:CHERRY_PLATE_100H, F.Cu at (197.6, 166.7)
- added SW3-8: MX, Keyboard:CHERRY_PLATE_100H, F.Cu at (216.7, 166.7)
- added SW3-9: MX, Keyboard:CHERRY_PLATE_100H, F.Cu at (235.7, 166.7)
- added SW4-10: MX, Keyboard:CHERRY_PLATE_125H, F.Cu at (242.9, 185.7)
- added SW4-11: MX, Keyboard:CHERRY_PLATE_100H, F.Cu at (264.3, 185.7)
- added SW4-12: MX, Keyboard:CHERRY_PLATE_125H, F.Cu at (285.8, 185.7)
- added SW4-13: MX, Keyboard:CHERRY_PLATE_100H, F.Cu at (307.2, 185.7)
- added SW4-14: MX, Keyboard:CHERRY_PLATE_100H, F.Cu at (326.2, 185.7)
- added SW4-15: MX, Keyboard:CHERRY_PLATE_100H, F.Cu at (345.3, 185.7)
- added SW4-2: MX, Keyboard:CHERRY_PLATE_150H, F.Cu at (97.6, 185.7)
- added SW4-7: MX, Keyboard:CHERRY_PLATE_625H, F.Cu at (171.4, 185.7)
- D0-0, D1-0, D2-0, D3-0, D4-0: moved to B.Cu
- SW0-0: footprint Keyboard:CHERRY_PCB_100H -> Keyboard:CHERRY_PLATE_100H
- SW1-0: footprint Keyboard:CHERRY_PCB_150H -> Keyboard:CHERRY_PLATE_150H
- SW2-0: footprint Keyboard:CHERRY_PCB_200H -> Keyboard:CHERRY_PLATE_175H
- SW3-0: footprint Keyboard:CHERRY_PCB_275H -> Keyboard:CHERRY_PLATE_225H
- SW4-0: footprint Keyboard:CHERRY_PLATE_150H -> Keyboard:CHERRY_PLATE_175H
- moved SW3-0 88.1 mm to (71.4, 166.7)
- moved SW2-0 85.9 mm to (66.7, 147.6)
- moved SW0-0 83.6 mm to (59.5, 109.5)
- moved SW1-0 83.6 mm to (64.3, 128.6)
- moved D0-0 82.2 mm to (54.8, 116.7), turned to 0 degrees
- moved SW4-0 81.4 mm to (66.7, 185.7)
- moved D1-0 77.9 mm to (59.5, 135.7), turned to 0 degrees
- moved D2-0 75.7 mm to (61.9, 154.8), turned to 0 degrees
- moved D4-0 75.7 mm to (61.9, 192.9), turned to 0 degrees
- moved D3-0 71.4 mm to (66.7, 173.8), turned to 0 degrees
Connections:
- D0-0 pad 1: Row-1 -> Col-0
- D1-0 pad 1: Row-2 -> Col-0
- D2-0 pad 1: Row-3 -> Col-0
- D3-0 pad 1: Row-4 -> Col-0
- SW0-0 pad 1: Row-0 -> Col-0
- SW1-0 pad 1: Row-1 -> Col-0
- SW2-0 pad 1: Row-2 -> Col-0
- SW3-0 pad 1: Row-3 -> Col-0
- SW4-0 pad 1: Row-4 -> Col-0
Other:
- board outline added: 315 x 104 mm

Commit message: Removes useless junctions
Connections:
- D0-1 pad 1: Col-0 -> Col-1
- D0-10 pad 1: Col-0 -> Col-10
- D0-11 pad 1: Col-0 -> Col-11
- D0-12 pad 1: Col-0 -> Col-12
- D0-14 pad 1: Col-0 -> Col-14
- D0-15 pad 1: Col-0 -> Col-15
- D0-2 pad 1: Col-0 -> Col-2
- D0-3 pad 1: Col-0 -> Col-3
- D0-4 pad 1: Col-0 -> Col-4
- D0-5 pad 1: Col-0 -> Col-5
- D0-6 pad 1: Col-0 -> Col-6
- D0-7 pad 1: Col-0 -> Col-7
- D0-8 pad 1: Col-0 -> Col-8
- D0-9 pad 1: Col-0 -> Col-9
- D1-1 pad 1: Col-0 -> Col-1
- D1-10 pad 1: Col-0 -> Col-10
- D1-11 pad 1: Col-0 -> Col-11
- D1-12 pad 1: Col-0 -> Col-12
- D1-14 pad 1: Col-0 -> Col-14
- D1-15 pad 1: Col-0 -> Col-15
- D1-2 pad 1: Col-0 -> Col-2
- D1-3 pad 1: Col-0 -> Col-3
- D1-4 pad 1: Col-0 -> Col-4
- D1-5 pad 1: Col-0 -> Col-5
- D1-6 pad 1: Col-0 -> Col-6
- D1-7 pad 1: Col-0 -> Col-7
- D1-8 pad 1: Col-0 -> Col-8
- D1-9 pad 1: Col-0 -> Col-9
- D2-1 pad 1: Col-0 -> Col-1
- D2-10 pad 1: Col-0 -> Col-10
- D2-11 pad 1: Col-0 -> Col-11
- D2-14 pad 1: Col-0 -> Col-14
- D2-15 pad 1: Col-0 -> Col-15
- D2-2 pad 1: Col-0 -> Col-2
- D2-3 pad 1: Col-0 -> Col-3
- D2-4 pad 1: Col-0 -> Col-4
- D2-5 pad 1: Col-0 -> Col-5
- D2-6 pad 1: Col-0 -> Col-6
- D2-7 pad 1: Col-0 -> Col-7
- D2-8 pad 1: Col-0 -> Col-8
- D2-9 pad 1: Col-0 -> Col-9
- D3-10 pad 1: Col-0 -> Col-10
- D3-11 pad 1: Col-0 -> Col-11
- D3-13 pad 1: Col-0 -> Col-13
- D3-14 pad 1: Col-0 -> Col-14
- D3-15 pad 1: Col-0 -> Col-15
- D3-2 pad 1: Col-0 -> Col-2
- D3-3 pad 1: Col-0 -> Col-3
- D3-4 pad 1: Col-0 -> Col-4
- D3-5 pad 1: Col-0 -> Col-5
- D3-6 pad 1: Col-0 -> Col-6
- D3-7 pad 1: Col-0 -> Col-7
- D3-8 pad 1: Col-0 -> Col-8
- D3-9 pad 1: Col-0 -> Col-9
- D4-10 pad 1: Col-0 -> Col-10
- D4-11 pad 1: Col-0 -> Col-11
- D4-12 pad 1: Col-0 -> Col-12
- D4-13 pad 1: Col-0 -> Col-13
- D4-14 pad 1: Col-0 -> Col-14
- D4-15 pad 1: Col-0 -> Col-15
- D4-2 pad 1: Col-0 -> Col-2
- D4-7 pad 1: Col-0 -> Col-7
- SW0-0 pad 1: Col-0 -> Row-0
- SW0-1 pad 1: Col-0 -> Row-0
- SW0-10 pad 1: Col-0 -> Row-0
- SW0-11 pad 1: Col-0 -> Row-0
- SW0-12 pad 1: Col-0 -> Row-0
- SW0-14 pad 1: Col-0 -> Row-0
- SW0-15 pad 1: Col-0 -> Row-0
- SW0-2 pad 1: Col-0 -> Row-0
- SW0-3 pad 1: Col-0 -> Row-0
- SW0-4 pad 1: Col-0 -> Row-0
- SW0-5 pad 1: Col-0 -> Row-0
- SW0-6 pad 1: Col-0 -> Row-0
- SW0-7 pad 1: Col-0 -> Row-0
- SW0-8 pad 1: Col-0 -> Row-0
- SW0-9 pad 1: Col-0 -> Row-0
- SW1-0 pad 1: Col-0 -> Row-1
- SW1-1 pad 1: Col-0 -> Row-1
- SW1-10 pad 1: Col-0 -> Row-1
- SW1-11 pad 1: Col-0 -> Row-1
- SW1-12 pad 1: Col-0 -> Row-1
- SW1-14 pad 1: Col-0 -> Row-1
- SW1-15 pad 1: Col-0 -> Row-1
- SW1-2 pad 1: Col-0 -> Row-1
- SW1-3 pad 1: Col-0 -> Row-1
- SW1-4 pad 1: Col-0 -> Row-1
- SW1-5 pad 1: Col-0 -> Row-1
- SW1-6 pad 1: Col-0 -> Row-1
- SW1-7 pad 1: Col-0 -> Row-1
- SW1-8 pad 1: Col-0 -> Row-1
- SW1-9 pad 1: Col-0 -> Row-1
- SW2-0 pad 1: Col-0 -> Row-2
- SW2-1 pad 1: Col-0 -> Row-2
- SW2-10 pad 1: Col-0 -> Row-2
- SW2-11 pad 1: Col-0 -> Row-2
- SW2-14 pad 1: Col-0 -> Row-2
- SW2-15 pad 1: Col-0 -> Row-2
- SW2-2 pad 1: Col-0 -> Row-2
- SW2-3 pad 1: Col-0 -> Row-2
- SW2-4 pad 1: Col-0 -> Row-2
- SW2-5 pad 1: Col-0 -> Row-2
- SW2-6 pad 1: Col-0 -> Row-2
- SW2-7 pad 1: Col-0 -> Row-2
- SW2-8 pad 1: Col-0 -> Row-2
- SW2-9 pad 1: Col-0 -> Row-2
- SW3-0 pad 1: Col-0 -> Row-3
- SW3-10 pad 1: Col-0 -> Row-3
- SW3-11 pad 1: Col-0 -> Row-3
- SW3-13 pad 1: Col-0 -> Row-3
- SW3-14 pad 1: Col-0 -> Row-3
- SW3-15 pad 1: Col-0 -> Row-3
- SW3-2 pad 1: Col-0 -> Row-3
- SW3-3 pad 1: Col-0 -> Row-3
- SW3-4 pad 1: Col-0 -> Row-3
- SW3-5 pad 1: Col-0 -> Row-3
- SW3-6 pad 1: Col-0 -> Row-3
- SW3-7 pad 1: Col-0 -> Row-3
- SW3-8 pad 1: Col-0 -> Row-3
- SW3-9 pad 1: Col-0 -> Row-3
- SW4-0 pad 1: Col-0 -> Row-4
- SW4-10 pad 1: Col-0 -> Row-4
- SW4-11 pad 1: Col-0 -> Row-4
- SW4-12 pad 1: Col-0 -> Row-4
- SW4-13 pad 1: Col-0 -> Row-4
- SW4-14 pad 1: Col-0 -> Row-4
- SW4-15 pad 1: Col-0 -> Row-4
- SW4-2 pad 1: Col-0 -> Row-4
- SW4-7 pad 1: Col-0 -> Row-4
